Commit message: updated instructions

File: openamrobot_description/urdf/robo_urdf.urdf.xacro (robot description, xacro)
@@ -28,19 +28,19 @@
       <geometry>
         <mesh
-          filename="package://omr_description/meshes/visual/base_link.STL" />
-      </geometry>
-      <material
-        name="">
-        <color
-          rgba="0.792156862745098 0.819607843137255 0.933333333333333 1" />
-      </material>
-    </visual>
-    <collision>
-      <origin
-        xyz="0 0 0"
-        rpy="0 0 0" />
-      <geometry>
-        <mesh
-          filename="package://omr_description/meshes/visual/base_link.STL" />
+          filename="package://openamrobot_description/meshes/visual/base_link.STL" />
+      </geometry>
+      <material
+        name="">
+        <color
+          rgba="0.792156862745098 0.819607843137255 0.933333333333333 1" />
+      </material>
+    </visual>
+    <collision>
+      <origin
+        xyz="0 0 0"
+        rpy="0 0 0" />
+      <geometry>
+        <mesh
+          filename="package://openamrobot_description/meshes/visual/base_link.STL" />
       </geometry>
     </collision>
@@ -68,19 +68,19 @@
       <geometry>
         <mesh
-          filename="package://omr_description/meshes/visual/fl_caster_link.STL" />
-      </geometry>
-      <material
-        name="">
-        <color
-          rgba="0.792156862745098 0.819607843137255 0.933333333333333 1" />
-      </material>
-    </visual>
-    <collision>
-      <origin
-        xyz="0 0 0"
-        rpy="0 0 0" />
-      <geometry>
-        <mesh
-          filename="package://omr_description/meshes/visual/fl_caster_link.STL" />
+          filename="package://openamrobot_description/meshes/visual/fl_caster_link.STL" />
+      </geometry>
+      <material
+        name="">
+        <color
+          rgba="0.792156862745098 0.819607843137255 0.933333333333333 1" />
+      </material>
+    </visual>
+    <collision>
+      <origin
+        xyz="0 0 0"
+        rpy="0 0 0" />
+      <geometry>
+        <mesh
+          filename="package://openamrobot_description/meshes/visual/fl_caster_link.STL" />
       </geometry>
     </collision>
@@ -122,5 +122,5 @@
       <geometry>
         <mesh
-          filename="package://omr_description/meshes/visual/fl_wheel_link.STL" />
+          filename="package://openamrobot_description/meshes/visual/fl_wheel_link.STL" />
       </geometry>
       <material
@@ -173,19 +173,19 @@
       <geometry>
         <mesh
-          filename="package://omr_description/meshes/visual/fr_caster_link.STL" />
-      </geometry>
-      <material
-        name="">
-        <color
-          rgba="0.792156862745098 0.819607843137255 0.933333333333333 1" />
-      </material>
-    </visual>
-    <collision>
-      <origin
-        xyz="0 0 0"
-        rpy="0 0 0" />
-      <geometry>
-        <mesh
-          filename="package://omr_description/meshes/visual/fr_caster_link.STL" />
+          filename="package://openamrobot_description/meshes/visual/fr_caster_link.STL" />
+      </geometry>
+      <material
+        name="">
+        <color
+          rgba="0.792156862745098 0.819607843137255 0.933333333333333 1" />
+      </material>
+    </visual>
+    <collision>
+      <origin
+        xyz="0 0 0"
+        rpy="0 0 0" />
+      <geometry>
+        <mesh
+          filename="package://openamrobot_description/meshes/visual/fr_caster_link.STL" />
       </geometry>
     </collision>
@@ -227,5 +227,5 @@
       <geometry>
         <mesh
-          filename="package://omr_description/meshes/visual/fr_wheel_link.STL" />
+          filename="package://openamrobot_description/meshes/visual/fr_wheel_link.STL" />
       </geometry>
       <material
@@ -278,19 +278,19 @@
       <geometry>
         <mesh
-          filename="package://omr_description/meshes/visual/br_caster_link.STL" />
-      </geometry>
-      <material
-        name="">
-        <color
-          rgba="0.792156862745098 0.819607843137255 0.933333333333333 1" />
-      </material>
-    </visual>
-    <collision>
-      <origin
-        xyz="0 0 0"
-        rpy="0 0 0" />
-      <geometry>
-        <mesh
-          filename="package://omr_description/meshes/visual/br_caster_link.STL" />
+          filename="package://openamrobot_description/meshes/visual/br_caster_link.STL" />
+      </geometry>
+      <material
+        name="">
+        <color
+          rgba="0.792156862745098 0.819607843137255 0.933333333333333 1" />
+      </material>
+    </visual>
+    <collision>
+      <origin
+        xyz="0 0 0"
+        rpy="0 0 0" />
+      <geometry>
+        <mesh
+          filename="package://openamrobot_description/meshes/visual/br_caster_link.STL" />
       </geometry>
     </collision>
@@ -332,5 +332,5 @@
       <geometry>
         <mesh
-          filename="package://omr_description/meshes/visual/br_wheel_link.STL" />
+          filename="package://openamrobot_description/meshes/visual/br_wheel_link.STL" />
       </geometry>
       <material
@@ -383,19 +383,19 @@
       <geometry>
         <mesh
-          filename="package://omr_description/meshes/visual/bl_caster_link.STL" />
-      </geometry>
-      <material
-        name="">
-        <color
-          rgba="0.792156862745098 0.819607843137255 0.933333333333333 1" />
-      </material>
-    </visual>
-    <collision>
-      <origin
-        xyz="0 0 0"
-        rpy="0 0 0" />
-      <geometry>
-        <mesh
-          filename="package://omr_description/meshes/visual/bl_caster_link.STL" />
+          filename="package://openamrobot_description/meshes/visual/bl_caster_link.STL" />
+      </geometry>
+      <material
+        name="">
+        <color
+          rgba="0.792156862745098 0.819607843137255 0.933333333333333 1" />
+      </material>
+    </visual>
+    <collision>
+      <origin
+        xyz="0 0 0"
+        rpy="0 0 0" />
+      <geometry>
+        <mesh
+          filename="package://openamrobot_description/meshes/visual/bl_caster_link.STL" />
       </geometry>
     </collision>
@@ -437,5 +437,5 @@
       <geometry>
         <mesh
-          filename="package://omr_description/meshes/visual/bl_wheel_link.STL" />
+          filename="package://openamrobot_description/meshes/visual/bl_wheel_link.STL" />
       </geometry>
       <material
@@ -488,5 +488,5 @@
       <geometry>
         <mesh
-          filename="package://omr_description/meshes/visual/left_wheel_link.STL" />
+          filename="package://openamrobot_description/meshes/visual/left_wheel_link.STL" />
       </geometry>
       <material
@@ -539,5 +539,5 @@
       <geometry>
         <mesh
-          filename="package://omr_description/meshes/visual/right_wheel_link.STL" />
+          filename="package://openamrobot_description/meshes/visual/right_wheel_link.STL" />
       </geometry>
       <material
@@ -590,19 +590,19 @@
       <geometry>
         <mesh
-          filename="package://omr_description/meshes/visual/lidar_link.STL" />
-      </geometry>
-      <material
-        name="">
-        <color
-          rgba="0.792156862745098 0.819607843137255 0.933333333333333 1" />
-      </material>
-    </visual>
-    <collision>
-      <origin
-        xyz="0 0 0"
-        rpy="0 0 0" />
-      <geometry>
-        <mesh
-          filename="package://omr_description/meshes/visual/lidar_link.STL" />
+          filename="package://openamrobot_description/meshes/visual/lidar_link.STL" />
+      </geometry>
+      <material
+        name="">
+        <color
+          rgba="0.792156862745098 0.819607843137255 0.933333333333333 1" />
+      </material>
+    </visual>
+    <collision>
+      <origin
+        xyz="0 0 0"
+        rpy="0 0 0" />
+      <geometry>
+        <mesh
+          filename="package://openamrobot_description/meshes/visual/lidar_link.STL" />
       </geometry>
     </collision>
